Commit message: fix effort & velocity limit

File: src/robot_urdf/urdf/robot_urdf.urdf (robot description, URDF)
Before this commit: robot AMR, 17 links, 16 joints
Joints:
- joint J1: limit lower=-4.7124 upper=4.7124 effort=150 velocity=3.15 -> lower=-4.7124 upper=4.7124 effort=2000 velocity=100
- joint J2: limit lower=-3.1416 upper=3.1416 effort=150 velocity=3.15 -> lower=-3.1416 upper=3.1416 effort=2000 velocity=100
- joint J3: limit lower=-3.1416 upper=3.1416 effort=150 velocity=3.15 -> lower=-3.1416 upper=3.1416 effort=2000 velocity=100
- joint J4: limit lower=-3.1416 upper=3.1416 effort=150 velocity=3.15 -> lower=-3.1416 upper=3.1416 effort=2000 velocity=100
- joint J5: limit lower=-3.1416 upper=3.1416 effort=150 velocity=3.15 -> lower=-3.1416 upper=3.1416 effort=2000 velocity=100
- joint J6: limit lower=-4.7124 upper=4.7124 effort=150 velocity=0 -> lower=-4.7124 upper=4.7124 effort=2000 velocity=100

Commit message: update tf script

File: src/robot_urdf/urdf/robot_urdf.urdf (robot description, URDF)
Before this commit: robot AMR, 17 links, 16 joints
Links:
- added link T265
- added link amr
Joints:
- added joint T265_trans: type fixed, parent base_link, child T265, origin xyz=-0.67365 0.14932  -0.31 rpy=1.57079632679 0 1.48352982679
- added joint amr_to_base_link: type fixed, parent amr, child base_link, origin xyz=-0.24888 0.15425 0.636 rpy=0 0 3.1415926535897
